File: proteusM54.kicad_pcb (KiCad board)
At the start: 2 copper layers, 154 x 160 mm, 21 parts, among them J1 Conn_01x01, J10 XH-10AW, J2 Conn_01x01, J3 Conn_01x06, J4 Conn_01x01, J5 Conn_01x01, J6 Conn_01x01, J9 7-967288-1, M2 Module-can-0.1, M3 Module-wbo-0.3, P1 Pad, U1 MPXxx6115A, U2 MPX4/MPXH6400_MAP

Commit message: Upd sch, pcb
Parts:
- added D1: D_Schottky, Diode_SMD:D_SMA, F.Cu at (194.0, 89.3)
- added D2: D_Schottky, Diode_SMD:D_SMA, F.Cu at (190.0, 89.3)
- added D3: D_Schottky, Diode_SMD:D_SMA, F.Cu at (180.0, 89.3)
- added D4: D_Schottky, Diode_SMD:D_SMA, F.Cu at (170.5, 89.3)
- added D5: D_Schottky, Diode_SMD:D_SMA, F.Cu at (160.5, 89.3)
- added F1: Fuse-Pad-Pad, hellen-one-common:PAD-1206-PAD, F.Cu at (221.5, 89.3)
- added F3: 10A, hellen-one-common:36911600000, F.Cu at (107.0, 96.3)
- added F4: 10A, hellen-one-common:36911600000, F.Cu at (122.0, 96.3)
- added F5: 10A, hellen-one-common:36911600000, F.Cu at (132.0, 96.3)
- added F6: 10A, hellen-one-common:36911600000, F.Cu at (117.0, 96.3)
- added F7: 10A, hellen-one-common:36911600000, F.Cu at (127.0, 96.3)
- added F8: 10A, hellen-one-common:36911600000, F.Cu at (112.0, 96.3)
- added P10: Pad, hellen-one-common:PAD-TH, F.Cu at (209.5, 92.3)
- added P11: Pad, hellen-one-common:PAD-TH, F.Cu at (206.5, 92.3)
- added P12: Pad, hellen-one-common:PAD-TH, F.Cu at (203.5, 92.3)
- added P13: Pad, hellen-one-common:PAD-TH, F.Cu at (200.5, 92.3)
- added P14: Pad, hellen-one-common:PAD-TH, F.Cu at (197.5, 92.3)
- added P15: Pad, hellen-one-common:PAD-TH, F.Cu at (212.5, 92.3)
- added P16: Pad, hellen-one-common:PAD-TH, F.Cu at (209.5, 87.8)
- added P17: Pad, hellen-one-common:PAD-TH, F.Cu at (206.5, 87.8)
- added P18: Pad, hellen-one-common:PAD-TH, F.Cu at (203.5, 87.8)
- added P19: Pad, hellen-one-common:PAD-TH, F.Cu at (200.5, 87.8)
- added P2: Pad, hellen-one-common:PAD-TH, F.Cu at (217.5, 92.3)
- added P20: Pad, hellen-one-common:PAD-TH, F.Cu at (197.5, 87.8)
- added P21: Pad, hellen-one-common:PAD-TH, F.Cu at (212.5, 87.8)
- added P22: Pad, hellen-one-common:PAD-TH, F.Cu at (186.5, 96.8)
- added P23: Pad, hellen-one-common:PAD-TH, F.Cu at (183.5, 87.8)
- added P24: Pad, hellen-one-common:PAD-TH, F.Cu at (180.0, 95.8)
- added P25: Pad, hellen-one-common:PAD-TH, F.Cu at (174.0, 87.8)
- added P26: Pad, hellen-one-common:PAD-TH, F.Cu at (167.0, 92.3)
- added P27: Pad, hellen-one-common:PAD-TH, F.Cu at (164.0, 92.3)
- added P28: Pad, hellen-one-common:PAD-TH, F.Cu at (160.5, 105.8)
- added P29: Pad, hellen-one-common:PAD-TH, F.Cu at (194.0, 95.8)
- added P3: Pad, hellen-one-common:PAD-TH, F.Cu at (228.0, 87.8)
- added P30: Pad, hellen-one-common:PAD-TH, F.Cu at (186.5, 92.3)
- added P31: Pad, hellen-one-common:PAD-TH, F.Cu at (160.5, 99.8)
- added P32: Pad, hellen-one-common:PAD-TH, F.Cu at (160.5, 96.8)
- added P33: Pad, hellen-one-common:PAD-TH, F.Cu at (186.5, 87.8)
- added P34: Pad, hellen-one-common:PAD-TH, F.Cu at (167.0, 87.8)
- added P35: Pad, hellen-one-common:PAD-TH, F.Cu at (164.0, 87.8)
- added P36: Pad, hellen-one-common:PAD-TH, F.Cu at (157.0, 99.8)
- added P37: Pad, hellen-one-common:PAD-TH, F.Cu at (154.0, 96.8)
- added P38: Pad, hellen-one-common:PAD-TH, F.Cu at (151.0, 92.3)
- added P39: Pad, hellen-one-common:PAD-TH, F.Cu at (148.0, 99.8)
- added P4: Pad, hellen-one-common:PAD-TH, F.Cu at (217.5, 87.8)
- added P40: Pad, hellen-one-common:PAD-TH, F.Cu at (145.0, 99.8)
- added P41: Pad, hellen-one-common:PAD-TH, F.Cu at (157.0, 96.8)
- added P42: Pad, hellen-one-common:PAD-TH, F.Cu at (148.0, 96.8)
- added P43: Pad, hellen-one-common:PAD-TH, F.Cu at (145.0, 95.3)
- added P44: Pad, hellen-one-common:PAD-TH, F.Cu at (142.0, 104.3)
- added P45: Pad, hellen-one-common:PAD-TH, F.Cu at (142.0, 95.3)
- added P46: Pad, hellen-one-common:PAD-TH, F.Cu at (139.0, 96.8)
- added P47: Pad, hellen-one-common:PAD-TH, F.Cu at (136.0, 96.8)
- added P48: Pad, hellen-one-common:PAD-TH, F.Cu at (157.0, 92.3)
- added P49: Pad, hellen-one-common:PAD-TH, F.Cu at (154.0, 92.3)
- added P5: Pad, hellen-one-common:PAD-TH, F.Cu at (212.5, 99.8)
- added P50: Pad, hellen-one-common:PAD-TH, F.Cu at (148.0, 92.3)
- added P51: Pad, hellen-one-common:PAD-TH, F.Cu at (142.0, 99.8)
- added P52: Pad, hellen-one-common:PAD-TH, F.Cu at (139.0, 92.3)
- added P53: Pad, hellen-one-common:PAD-TH, F.Cu at (136.0, 92.3)
- added P54: Pad, hellen-one-common:PAD-TH, F.Cu at (157.0, 87.8)
- added P55: Pad, hellen-one-common:PAD-TH, F.Cu at (154.0, 87.8)
- added P56: Pad, hellen-one-common:PAD-TH, F.Cu at (151.0, 96.8)
- added P57: Pad, hellen-one-common:PAD-TH, F.Cu at (151.0, 87.8)
- added P58: Pad, hellen-one-common:PAD-TH, F.Cu at (148.0, 87.8)
- added P59: Pad, hellen-one-common:PAD-TH, F.Cu at (139.0, 87.8)
- added P6: Pad, hellen-one-common:PAD-TH, F.Cu at (209.5, 96.8)
- added P60: Pad, hellen-one-common:PAD-TH, F.Cu at (136.0, 87.8)
- added P61: Pad, hellen-one-common:PAD-TH, F.Cu at (121.5, 87.8)
- added P62: Pad, hellen-one-common:PAD-TH, F.Cu at (129.5, 87.8)
- added P7: Pad, hellen-one-common:PAD-TH, F.Cu at (200.5, 96.8)
- added P8: Pad, hellen-one-common:PAD-TH, F.Cu at (197.5, 96.8)
- added P9: Pad, hellen-one-common:PAD-TH, F.Cu at (212.5, 96.8)
- added Q1: ISL9V3040S3S, Package_TO_SOT_SMD:TO-263-2, F.Cu at (179.4, -43.4)
- added Q2: ISL9V3040S3S, Package_TO_SOT_SMD:TO-263-2, F.Cu at (143.5, -65.8)
- added Q3: ISL9V3040S3S, Package_TO_SOT_SMD:TO-263-2, F.Cu at (161.7, -43.4)
- added Q4: ISL9V3040S3S, Package_TO_SOT_SMD:TO-263-2, F.Cu at (147.0, 125.7)
- added Q5: ISL9V3040S3S, Package_TO_SOT_SMD:TO-263-2, F.Cu at (161.7, -31.1)
- added Q6: ISL9V3040S3S, Package_TO_SOT_SMD:TO-263-2, F.Cu at (144.1, -31.1)
- added Q7: AUIPS2041LTR, Package_TO_SOT_SMD:SOT-223, F.Cu at (173.5, 96.8)
- added R1: Jumper-Pad-Pad, hellen-one-common:PAD-0805-PAD, F.Cu at (142.0, 89.3)
- added R10: DNP, Resistor_SMD:R_2512_6332Metric, F.Cu at (139.6, -1.83)
- added R11: DNP, Resistor_SMD:R_2512_6332Metric, F.Cu at (174.9, -29.6)
- added R12: DNP, Resistor_SMD:R_2512_6332Metric, F.Cu at (159.1, -12.0)
- added R13: DNP, Resistor_SMD:R_2512_6332Metric, F.Cu at (166.9, -17.5)
- added R14: DNP, Resistor_SMD:R_2512_6332Metric, F.Cu at (166.9, -22.4)
- added R15: DNP, Resistor_SMD:R_2512_6332Metric, F.Cu at (184.6, -34.8)
- added R16: 10k, Resistor_SMD:R_0402_1005Metric, F.Cu at (201.1, -28.3)
- added R2: 22, hellen-one-common:R0603, F.Cu at (155.5, -0.28)
- added R3: 22, hellen-one-common:R0603, F.Cu at (152.2, -1.15)
- added R4: 22, hellen-one-common:R0603, F.Cu at (210.0, -37.3)
- added R7: 22, hellen-one-common:R0603, F.Cu at (166.5, -3.70)
- added R8: 22, hellen-one-common:R0603, F.Cu at (180.2, -7.15)
- added R9: 22, hellen-one-common:R0603, F.Cu at (213.8, -41.0)
- moved U2 403.5 mm to (141.9, 202.2), turned to 180 degrees
- moved U1 382.5 mm to (111.4, 191.9), turned to 180 degrees
- moved R5 364.0 mm to (123.1, 189.3), turned to -90 degrees
- moved C4 361.7 mm to (157.6, 186.4), turned to 90 degrees
- moved J10 320.3 mm to (161.2, 199.4)
- moved M2 275.8 mm to (239.2, 203.6), turned to 90 degrees
- moved M3 264.4 mm to (228.6, 189.0), turned to 180 degrees
- moved J3 261.5 mm to (213.9, 186.7), turned to 90 degrees
- moved P1 247.2 mm to (225.0, 87.8)
- moved C1 218.6 mm to (123.1, 192.4), turned to -90 degrees
- moved F2 213.1 mm to (145.0, 88.8), turned to -90 degrees
- moved C2 211.5 mm to (126.7, 189.2), turned to 90 degrees
- moved R6 186.4 mm to (155.3, 186.4), turned to -90 degrees
- moved C3 183.1 mm to (155.1, 192.0), turned to -90 degrees
- moved BRD1 0.39 mm to (239.8, 101.4)
Connections:
- F2 pad 1: unconnected-(F2-Pad1) -> Net-(J9-PadD26)
- F2 pad 2: /12V_MR -> /12V_IGN
- J3 pad 6: (no net) -> unconnected-(J3-Pad6)
- J9 pad A1: (no net) -> /OUT_INJ_RELAY
- J9 pad A2: (no net) -> Net-(J9-PadA2)
- J9 pad A3: (no net) -> Net-(J9-PadA3)
- J9 pad A4: (no net) -> GND
- J9 pad A5: (no net) -> GND
- J9 pad A6: (no net) -> GND
- J9 pad A7: (no net) -> Net-(J9-PadA7)
- J9 pad A8: (no net) -> Net-(J9-PadA8)
- J9 pad A9: (no net) -> Net-(J9-PadA9)
- J9 pad B1: (no net) -> Net-(J9-PadB1)
- J9 pad B10: (no net) -> Net-(J9-PadB10)
- J9 pad B11: (no net) -> Net-(J9-PadB11)
- J9 pad B12: (no net) -> Net-(J9-PadB12)
- J9 pad B13: (no net) -> Net-(J9-PadB13)
- J9 pad B14: (no net) -> Net-(J9-PadB14)
- J9 pad B15: (no net) -> Net-(J9-PadB15)
- J9 pad B16: (no net) -> Net-(J9-PadB16)
- J9 pad B17: (no net) -> Net-(J9-PadB17)
- J9 pad B18: (no net) -> Net-(J9-PadB18)
- J9 pad B19: (no net) -> Net-(J9-PadB19)
- J9 pad B2: (no net) -> Net-(J9-PadB2)
- J9 pad B20: (no net) -> GND
- J9 pad B21: (no net) -> GND
- J9 pad B22: (no net) -> GND
- J9 pad B23: (no net) -> /OUT_MAIN_RELAY
- J9 pad B24: (no net) -> GND
- J9 pad B3: (no net) -> /CAN_L
- J9 pad B4: (no net) -> /CAN_H
- J9 pad B5: (no net) -> Net-(J9-PadB5)
- J9 pad B6: (no net) -> Net-(J9-PadB6)
- J9 pad B7: (no net) -> Net-(J9-PadB7)
- J9 pad B8: (no net) -> Net-(J9-PadB8)
- J9 pad B9: (no net) -> Net-(J9-PadB9)
- J9 pad C1: (no net) -> /IN_MAF
- J9 pad C10: (no net) -> /IN_TPS2
- J9 pad C11: (no net) -> Net-(J9-PadC11)
- J9 pad C12: (no net) -> Net-(J9-PadC12)
- J9 pad C13: (no net) -> Net-(J9-PadC13)
- J9 pad C14: (no net) -> Net-(J9-PadC14)
- J9 pad C15: (no net) -> GND
- J9 pad C16: (no net) -> Net-(J9-PadC16)
- J9 pad C17: (no net) -> GND
- J9 pad C18: (no net) -> GND
- J9 pad C19: (no net) -> /IN_TPS1
- J9 pad C2: (no net) -> /IN_CAM2
- J9 pad C20: (no net) -> GND
- J9 pad C21: (no net) -> GND
- J9 pad C22: (no net) -> /IN_IAT
- J9 pad C23: (no net) -> GND
- J9 pad C24: (no net) -> /IN_CLT
- J9 pad C25: (no net) -> GND
- J9 pad C26: (no net) -> Net-(J9-PadC26)
- J9 pad C27: (no net) -> /IN_OILT
- J9 pad C28: (no net) -> GND
- J9 pad C29: (no net) -> /IN_KNOCK1
- J9 pad C3: (no net) -> Net-(J9-PadC3)
- J9 pad C30: (no net) -> GND
- J9 pad C31: (no net) -> /IN_KNOCK2
- J9 pad C32: (no net) -> GND
- J9 pad C33: (no net) -> /OUT_INJ1
- J9 pad C34: (no net) -> /OUT_INJ2
- J9 pad C35: (no net) -> /OUT_INJ3
- J9 pad C36: (no net) -> /OUT_INJ4
- J9 pad C37: (no net) -> /OUT_INJ5
- J9 pad C38: (no net) -> /OUT_INJ6
- J9 pad C39: (no net) -> Net-(J9-PadC39)
- J9 pad C4: (no net) -> Net-(J9-PadC4)
- J9 pad C40: (no net) -> /OUT_VANOS_INTAKE
- J9 pad C41: (no net) -> /OUT_VANOS_EXHAUST
- J9 pad C42: (no net) -> Net-(J9-PadC42)
- J9 pad C43: (no net) -> /OUT_ETB1
- J9 pad C44: (no net) -> /OUT_ETB2
- J9 pad C45: (no net) -> /OUT_MAP_THERMOSTAT
- J9 pad C46: (no net) -> /OUT_IDLE_CLOSE
- J9 pad C47: (no net) -> /OUT_IDLE_OPEN
- J9 pad C48: (no net) -> GND
- J9 pad C49: (no net) -> /OUT_INTAKE_VALVE
- J9 pad C5: (no net) -> /IN_CAM1
- J9 pad C50: (no net) -> Net-(J9-PadC50)
- J9 pad C51: (no net) -> Net-(J9-PadC51)
- J9 pad C52: (no net) -> /OUT_SEC_AIR_PUMP_VALVE
- J9 pad C6: (no net) -> Net-(J9-PadC6)
- J9 pad C7: (no net) -> +5VA
- J9 pad C8: (no net) -> /IN_CRANK
- J9 pad C9: (no net) -> Net-(J9-PadC9)
- J9 pad D1: (no net) -> Net-(J9-PadD1)
- J9 pad D10: (no net) -> /OUT_FUEL_PUMP_RELAY
- J9 pad D11: (no net) -> Net-(J9-PadD11)
- J9 pad D12: (no net) -> GND
- J9 pad D13: (no net) -> /IN_PPS2
- J9 pad D14: (no net) -> +5VA
- J9 pad D15: (no net) -> Net-(J9-PadD15)
- J9 pad D16: (no net) -> Net-(J9-PadD16)
- J9 pad D17: (no net) -> Net-(J9-PadD17)
- J9 pad D18: (no net) -> Net-(J9-PadD18)
- J9 pad D19: (no net) -> Net-(J9-PadD19)
- J9 pad D2: (no net) -> Net-(J9-PadD2)
- J9 pad D20: (no net) -> Net-(J9-PadD20)
- J9 pad D21: (no net) -> Net-(J9-PadD21)
- J9 pad D22: (no net) -> Net-(J9-PadD22)
- J9 pad D23: (no net) -> /IN_CLUTCH
- J9 pad D24: (no net) -> /IN_BRAKE
- J9 pad D25: (no net) -> Net-(J9-PadD25)
- J9 pad D26: (no net) -> Net-(J9-PadD26)
- J9 pad D27: (no net) -> Net-(J9-PadD27)
- J9 pad D28: (no net) -> /IN_BRAKE2
- J9 pad D29: (no net) -> Net-(J9-PadD29)
- J9 pad D3: (no net) -> /OUT_SEC_AIR_PUMP_RELAY
- J9 pad D30: (no net) -> Net-(J9-PadD30)
- J9 pad D31: (no net) -> Net-(J9-PadD31)
- J9 pad D32: (no net) -> Net-(J9-PadD32)
- J9 pad D33: (no net) -> Net-(J9-PadD33)
- J9 pad D34: (no net) -> Net-(J9-PadD34)
- J9 pad D35: (no net) -> Net-(J9-PadD35)
- J9 pad D36: (no net) -> /CAN2_H
- J9 pad D37: (no net) -> /CAN2_L
- J9 pad D38: (no net) -> Net-(J9-PadD38)
- J9 pad D39: (no net) -> Net-(J9-PadD39)
- J9 pad D4: (no net) -> Net-(J9-PadD4)
- J9 pad D40: (no net) -> Net-(J9-PadD40)
- J9 pad D5: (no net) -> Net-(J9-PadD5)
- J9 pad D6: (no net) -> Net-(J9-PadD6)
- J9 pad D7: (no net) -> GND
- J9 pad D8: (no net) -> /IN_PPS1
- J9 pad D9: (no net) -> +5VA
- J9 pad E1: (no net) -> /HV3
- J9 pad E2: (no net) -> /HV2
- J9 pad E3: (no net) -> /HV1
- J9 pad E4: (no net) -> Net-(J9-PadE4)
- J9 pad E5: (no net) -> GND
- J9 pad E6: (no net) -> /HV6
- J9 pad E7: (no net) -> /HV5
- J9 pad E8: (no net) -> Net-(J9-PadE8)
- J9 pad E9: (no net) -> /HV4
- J9 pad MH1: (no net) -> unconnected-(J9-PadMH1)
- J9 pad MH2: (no net) -> unconnected-(J9-PadMH2)
- J9 pad MH3: (no net) -> unconnected-(J9-PadMH3)
- J9 pad MH4: (no net) -> unconnected-(J9-PadMH4)
- M2 pad S1: (no net) -> /CAN_L
- M2 pad S2: (no net) -> /CAN_H
- M3 pad J2: (no net) -> unconnected-(M3-PadJ2)
- M3 pad J_GND2: (no net) -> unconnected-(M3-PadJ_GND2)
- M3 pad J_VCC1: (no net) -> unconnected-(M3-PadJ_VCC1)
- M3 pad J_VCC2: (no net) -> unconnected-(M3-PadJ_VCC2)
- P1 pad 1: (no net) -> Net-(J9-PadA2)
- U2 pad 4: (no net) -> unconnected-(U2-Pad4)
- U2 pad 5: (no net) -> unconnected-(U2-Pad5)
- U2 pad 6: (no net) -> unconnected-(U2-Pad6)

Commit message: Upd pcb
Parts:
- added G***: LOGO, LOGO, F.Cu at (251.2, 137.8)
- added G1: RUSEFI_LOGO, kicad6-libraries:rusefi_logo, F.Cu at (255.0, 202.6)
- added G2: PROTO_AREA, hellen-one-common:PROTO_AREA, F.Cu at (256.3, 117.5)
- added G3: PROTO_AREA, hellen-one-common:PROTO_AREA, F.Cu at (248.7, 117.5)
- added G4: PROTO_AREA, hellen-one-common:PROTO_AREA, F.Cu at (241.1, 117.5)
- added G5: PROTO_AREA, hellen-one-common:PROTO_AREA, F.Cu at (248.7, 104.8)
- added G6: PROTO_AREA, hellen-one-common:PROTO_AREA, F.Cu at (256.3, 125.1)
- added G7: PROTO_AREA, hellen-one-common:PROTO_AREA, F.Cu at (241.1, 104.8)
- added G8: PROTO_AREA, hellen-one-common:PROTO_AREA, F.Cu at (256.3, 104.8)
- added J7: Conn_01x01, TestPoint:TestPoint_Pad_D4.0mm, B.Cu at (234.7, 95.9)
- added P63: Pad, hellen-one-common:PAD-TH, F.Cu at (204.2, 146.6)
- added P64: Pad, hellen-one-common:PAD-TH, F.Cu at (204.5, 160.0)
- added P65: Pad, hellen-one-common:PAD-TH, F.Cu at (204.5, 168.9)
- added P66: Pad, hellen-one-common:PAD-TH, F.Cu at (204.5, 164.5)
- added P67: Pad, hellen-one-common:PAD-TH, F.Cu at (204.5, 155.5)
- added P68: Pad, hellen-one-common:PAD-TH, F.Cu at (204.2, 137.4)
- added P69: Pad, hellen-one-common:PAD-TH, F.Cu at (204.2, 140.4)
- added P70: Pad, hellen-one-common:PAD-TH, F.Cu at (204.2, 143.3)
- added P71: Pad, hellen-one-common:PAD-TH, F.Cu at (204.5, 151.1)
- added P72: Pad, hellen-one-common:PAD-TH, F.Cu at (176.3, 185.3)
- added P73: Pad, hellen-one-common:PAD-TH, F.Cu at (179.2, 185.3)
- added P74: Pad, hellen-one-common:PAD-TH, F.Cu at (170.2, 185.3)
- added P75: Pad, hellen-one-common:PAD-TH, F.Cu at (173.2, 185.3)
- added P76: Pad, hellen-one-common:PAD-TH, F.Cu at (183.4, 185.3)
- added P77: Pad, hellen-one-common:PAD-TH, F.Cu at (186.4, 185.3)
- added P78: Pad, hellen-one-common:PAD-TH, F.Cu at (140.2, 131.4)
- added P79: Pad, hellen-one-common:PAD-TH, F.Cu at (140.2, 137.5)
- added P80: Pad, hellen-one-common:PAD-TH, F.Cu at (140.2, 134.5)
- added P81: Pad, hellen-one-common:PAD-TH, F.Cu at (140.2, 140.6)
- added P82: Pad, hellen-one-common:PAD-TH, F.Cu at (140.2, 147.2)
- added P83: Pad, hellen-one-common:PAD-TH, F.Cu at (140.1, 155.3)
- moved R4 254.6 mm to (83.2, 183.6), turned to 90 degrees
- moved Q3 244.1 mm to (92.2, 190.6)
- moved R9 219.6 mm to (83.2, 135.6), turned to 90 degrees
- moved Q5 217.1 mm to (92.2, 174.6)
- moved R12 207.1 mm to (88.2, 182.6)
- moved R14 204.8 mm to (88.2, 166.6)
- moved R8 199.9 mm to (83.2, 167.6), turned to 90 degrees
- moved R15 194.9 mm to (88.2, 134.6)
- moved Q1 191.1 mm to (92.2, 126.6)
- moved R13 185.6 mm to (88.2, 150.6)
- moved Q2 183.7 mm to (92.2, 110.6), turned to 0 degrees
- moved Q6 181.2 mm to (92.2, 142.6)
- moved R7 176.2 mm to (83.2, 151.6), turned to 90 degrees
- moved R11 158.1 mm to (88.2, 102.6)
- moved R2 140.0 mm to (83.2, 119.6), turned to 90 degrees
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Connections:
- BRD1 pad A1(12): unconnected-(BRD1-PadA1(12)) -> Net-(BRD1-PadA1(12))
- BRD1 pad A13(23): unconnected-(BRD1-PadA13(23)) -> Net-(BRD1-PadA13(23))
- BRD1 pad A14(22): unconnected-(BRD1-PadA14(22)) -> Net-(BRD1-PadA14(22))
- BRD1 pad A2(11): unconnected-(BRD1-PadA2(11)) -> Net-(BRD1-PadA2(11))
- BRD1 pad A26(33): unconnected-(BRD1-PadA26(33)) -> Net-(BRD1-PadA26(33))
- BRD1 pad A27(32): unconnected-(BRD1-PadA27(32)) -> Net-(P63-Pad1)
- BRD1 pad A28(31): unconnected-(BRD1-PadA28(31)) -> Net-(BRD1-PadA28(31))
- BRD1 pad A29(30): unconnected-(BRD1-PadA29(30)) -> Net-(BRD1-PadA29(30))
- BRD1 pad A30(29): unconnected-(BRD1-PadA30(29)) -> Net-(BRD1-PadA30(29))
- BRD1 pad B12(12): unconnected-(BRD1-PadB12(12)) -> Net-(BRD1-PadB12(12))
- BRD1 pad B13(11): unconnected-(BRD1-PadB13(11)) -> Net-(BRD1-PadB13(11))
- BRD1 pad B15(9): unconnected-(BRD1-PadB15(9)) -> Net-(BRD1-PadB15(9))
- BRD1 pad B4(5): unconnected-(BRD1-PadB4(5)) -> Net-(BRD1-PadB4(5))
- BRD1 pad B5(4): unconnected-(BRD1-PadB5(4)) -> Net-(BRD1-PadB5(4))
- BRD1 pad B8(1): unconnected-(BRD1-PadB8(1)) -> Net-(BRD1-PadB8(1))
- BRD1 pad C10(3): unconnected-(BRD1-PadC10(3)) -> Net-(BRD1-PadC22(14))
- BRD1 pad C11(2): unconnected-(BRD1-PadC11(2)) -> /12V_PROT
- BRD1 pad C12(1): unconnected-(BRD1-PadC12(1)) -> /12V_PROT
- BRD1 pad C17(19): unconnected-(BRD1-PadC17(19)) -> Net-(BRD1-PadC17(19))
- BRD1 pad C18(18): unconnected-(BRD1-PadC18(18)) -> Net-(BRD1-PadC18(18))
- BRD1 pad C22(14): unconnected-(BRD1-PadC22(14)) -> Net-(BRD1-PadC22(14))
- BRD1 pad C27(32): unconnected-(BRD1-PadC27(32)) -> Net-(BRD1-PadC27(32))
- BRD1 pad C28(31): unconnected-(BRD1-PadC28(31)) -> Net-(BRD1-PadC28(31))
- BRD1 pad C31(28): unconnected-(BRD1-PadC31(28)) -> Net-(BRD1-PadC31(28))
- BRD1 pad C33(26): unconnected-(BRD1-PadC33(26)) -> Net-(BRD1-PadC22(14))
Routing:
- net +5VA: track 0.00 -> 435.6 mm, vias 0 -> 3
- net /12V_MR: track 0.00 -> 297.8 mm
- net /12V_PROT: track 0.00 -> 274.2 mm
- net /CAN_L: track 0.00 -> 270.3 mm, vias 0 -> 2
- net /CAN_H: track 0.00 -> 259.1 mm, vias 0 -> 2
- net /GATE_IGN3: track 0.00 -> 197.3 mm, vias 0 -> 1
- net /GATE_IGN5: track 0.00 -> 174.3 mm, vias 0 -> 1
- net /OUT_FUEL_PUMP_RELAY: track 0.00 -> 166.7 mm, vias 0 -> 1
- net /OUT_INJ2: track 0.00 -> 162.4 mm, vias 0 -> 1
- net /GATE_IGN4: track 0.00 -> 160.3 mm, vias 0 -> 1
- net /OUT_INJ3: track 0.00 -> 159.7 mm, vias 0 -> 1
- net /GATE_IGN2: track 0.00 -> 156.4 mm, vias 0 -> 1
- net /OUT_INJ4: track 0.00 -> 149.6 mm, vias 0 -> 1
- net /OUT_INJ5: track 0.00 -> 144.0 mm, vias 0 -> 1
- net /IN_KNOCK1: track 0.00 -> 142.3 mm, vias 0 -> 1
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- added copper zone on In1.Cu, net GND
- added copper zone on In2.Cu, net GND
Other:
- board size 154 x 160 mm -> 182 x 160 mm
- copper layers 2 -> 4
- board text added: "+12 +5 GND"
- board text added: "BARO"
- board text added: "GND"
- board text added: "GND GND H- H- Rtrim Ip Vs/Ip VS H+ H+"
- board text added: "Proteus BMW M54 adapter rev. a"
- board text added: "SWD: V C G D R"
- board text added: "WBO"
- board text added: "https://rusefi.com/s/proteus-m54"
