File: proteusM54.kicad_sch (KiCad schematic)
At the start: 68 parts, among them J1 Conn_01x01, J10 XH-10AW, J12 XH-10A, J2 Conn_01x01, J3 Conn_01x06, J4 Conn_01x01, J5 Conn_01x01, J6 Conn_01x01, J9 7-967288-1, M2 Module-can-0.1, M3 Module-wbo-0.3, U1 MPXxx6115A, U2 MPX4/MPXH6400_MAP

Commit message: Upd sch, pcb
Parts:
- removed P? (x3): Pad, hellen-one-common:PAD-TH, symbol hellen-one-common:Pad
- added D1, D2, D3, D4, D5: D_Schottky, Diode_SMD:D_SMA, symbol Device:D_Schottky
- added P1, P10, P11, P12, P13, P14, P19, P2, P22, P23, P24, P25, P26, P27, P28, P29, P30, P31, P32, P34, P36, P37, P39, P4, P40, P41, P42, P43, P45, P46, P48, P50, P51, P52, P54, P57, P58, P59, P6, P60, P61, P62, P7: Pad, hellen-one-common:PAD-TH, symbol hellen-one-common:Pad
- added Q7: AUIPS2041LTR, Package_TO_SOT_SMD:SOT-223, symbol Power_Management:AUIPS2041L
- added R1: Jumper-Pad-Pad, hellen-one-common:PAD-0805-PAD, symbol hellen-one-common:Jumper-Pad-Pad
- added R16: 10k, Resistor_SMD:R_0402_1005Metric, symbol Device:R
- gave numbers to parts that had none: 45
Connections:
- net +5VA: now also BRD1.C21(15) (5V_1), BRD1.C32(27) (5V_1), BRD1.C9(4) (5V_1); no longer BRD1.C21 (5V_1), BRD1.C32 (5V_1), BRD1.C9 (5V_1)
- net 12V_IGN: now also BRD1.B18(21) (12V_IGN); no longer BRD1.B18 (12V_IGN)
- net 12V_MR: now also BRD1.B23(16) (12V_MR), D1.1 (K), D2.1 (K), D3.1 (K), D4.1 (K), D5.1 (K); no longer BRD1.B23 (12V_MR)
- net CAN2_H: now also BRD1.B22(17) (CAN2+); no longer BRD1.B22 (CAN2+)
- net CAN2_L: now also BRD1.B21(18) (CAN2-); no longer BRD1.B21 (CAN2-)
- net CAN_H: now also BRD1.B17(22) (CAN+); no longer BRD1.B17 (CAN+)
- net CAN_L: now also BRD1.B16(23) (CAN-); no longer BRD1.B16 (CAN-)
- net GATE_IGN1: now also BRD1.A35(24) (IGN1); no longer BRD1.A35 (IGN1)
- net GATE_IGN2: now also BRD1.A34(25) (IGN2); no longer BRD1.A34 (IGN2)
- net GATE_IGN3: now also BRD1.A22(14) (IGN3); no longer BRD1.A22 (IGN3)
- net GATE_IGN4: now also BRD1.A33(26) (IGN4); no longer BRD1.A33 (IGN4)
- net GATE_IGN5: now also BRD1.A32(27) (IGN5); no longer BRD1.A32 (IGN5)
- net GATE_IGN6: now also BRD1.A31(28) (IGN6); no longer BRD1.A31 (IGN6)
- net GND: now also BRD1.A17(19) (GND), BRD1.A18(18) (GND), BRD1.A24(35) (GND), BRD1.B14(10) (GND), BRD1.B19(20) (GND), BRD1.B20(19) (GND), BRD1.C1(12) (GND_SENS), BRD1.C2(11) (GND_SENS), BRD1.C23(13) (GND_SENS), BRD1.C29(30) (GND_SENS), BRD1.C3(10) (GND_SENS), BRD1.C4(9) (GND_SENS), BRD1.C5(8) (GND_SENS), BRD1.C6(7) (GND_SENS), BRD1.C7(6) (GND_SENS), BRD1.C8(5) (GND_SENS), Q7.3 (S), R1.2, R16.1; no longer BRD1.A17 (GND), BRD1.A18 (GND), BRD1.A24 (GND), BRD1.B14 (GND), BRD1.B19 (GND), BRD1.B20 (GND), BRD1.C1 (GND_SENS), BRD1.C2 (GND_SENS), BRD1.C23 (GND_SENS), BRD1.C29 (GND_SENS), BRD1.C3 (GND_SENS), BRD1.C4 (GND_SENS), BRD1.C5 (GND_SENS), BRD1.C6 (GND_SENS), BRD1.C7 (GND_SENS), BRD1.C8 (GND_SENS)
- net HV1: now also J9.E3; no longer J9.E1
- net HV3: now also J9.E1; no longer J9.E3
- net HV5: now also J9.E7; no longer J9.E6
- net HV6: now also J9.E6; no longer J9.E7
- net IN_BARO: now also BRD1.C26(33) (AV6)
- net IN_BRAKE: now also BRD1.B3(6) (D4); no longer BRD1.B3 (D4)
- net IN_BRAKE2: now also BRD1.B9(15) (D5); no longer BRD1.B9 (D5)
- net IN_CAM1: now also BRD1.B10(14) (D1); no longer BRD1.B10 (D1)
- net IN_CAM2: now also BRD1.B1(8) (D2); no longer BRD1.B1 (D2)
- net IN_CLT: now also BRD1.C20(16) (AT3(CLT)); no longer BRD1.C30 (AT2)
- net IN_CLUTCH: now also BRD1.B11(13) (D6); no longer BRD1.B11 (D6)
- net IN_CRANK: now also BRD1.B2(7) (D3); no longer BRD1.B2 (D3)
- net IN_IAT: now also BRD1.C30(29) (AT2(IAT)); no longer BRD1.C19 (AT1)
- net IN_KNOCK1: now also BRD1.C34(25) (KNOCK1); no longer BRD1.C34 (KNOCK1)
- net IN_KNOCK2: now also BRD1.C35(24) (KNOCK2); no longer BRD1.C35 (KNOCK2)
- net IN_MAF: now also BRD1.C16(20) (AV7); no longer BRD1.C13 (AV1)
- net IN_MAP: now also BRD1.C13(23) (AV1(MAP))
- net IN_OILT: now also BRD1.C19(17) (AT1); no longer BRD1.C20 (AT3)
- net IN_PPS1: now also BRD1.C25(34) (AV4); no longer BRD1.C25 (AV4)
- net IN_PPS2: now also BRD1.C15(21) (AV5); no longer BRD1.C15 (AV5)
- net IN_TPS1: now also BRD1.C24(35) (AV2(TPS)), J9.C19; no longer BRD1.C24 (AV2), J9.C10
- net IN_TPS2: now also BRD1.C14(22) (AV3), J9.C10; no longer BRD1.C14 (AV3), J9.C19
- net OUT_ETB1: now also BRD1.B7(2) (ETB1+); no longer BRD1.B7 (ETB1+)
- net OUT_ETB2: now also BRD1.B6(3) (ETB1-); no longer BRD1.B6 (ETB1-)
- net OUT_FUEL_PUMP_RELAY: now also BRD1.A8(5) (LS9(INJ9)); no longer BRD1.A8 (LS9)
- net OUT_IDLE_CLOSE: now also BRD1.A12(1) (LS15(FAN)); no longer BRD1.A12 (LS15)
- net OUT_IDLE_OPEN: now also BRD1.A23(13) (LS16(FUEL)); no longer BRD1.A23 (LS16)
- net OUT_INJ1: now also BRD1.A3(10) (LS1(INJ1)); no longer BRD1.A4 (LS3)
- net OUT_INJ2: now also BRD1.A15(21) (LS2(INJ2)); no longer BRD1.A16 (LS4)
- net OUT_INJ3: now also BRD1.A4(9) (LS3(INJ3)); no longer BRD1.A5 (LS5)
- net OUT_INJ4: now also BRD1.A16(20) (LS4(INJ4)); no longer BRD1.A6 (LS6)
- net OUT_INJ5: now also BRD1.A5(8) (LS5(INJ5)); no longer BRD1.A7 (LS7)
- net OUT_INJ6: now also BRD1.A6(7) (LS6(INJ6)); no longer BRD1.A19 (LS8)
- net OUT_INJ_RELAY: now also BRD1.A7(6) (LS7(INJ7)); no longer BRD1.A3 (LS1)
- net OUT_INTAKE_VALVE: now also BRD1.A10(3) (LS13(MAIN)), D4.2 (A)
- net OUT_MAIN_RELAY: now also BRD1.A19(17) (LS8(INJ8)); no longer BRD1.A15 (LS2)
- net OUT_MAP_THERMOSTAT: now also BRD1.A21(15) (LS12(INJ12)), D3.2 (A)
- net OUT_SEC_AIR_PUMP_RELAY: now also Q7.2 (D)
- net OUT_SEC_AIR_PUMP_VALVE: now also BRD1.A11(2) (LS14), D5.2 (A)
- net at J9.D39: now also P59.1 (Pin_1)
- net at J9.D38: now also R1.1
- net at J9.A2: now also P1.1 (Pin_1)
- net at J9.A3: now also P2.1 (Pin_1)
- net at J9.A9: now also P4.1 (Pin_1)
- net at J9.B10: now also P12.1 (Pin_1)
- net at J9.B11: now also P13.1 (Pin_1)
- net at J9.B12: now also P14.1 (Pin_1)
- net at J9.B17: now also P19.1 (Pin_1)
- net at J9.B2: now also P6.1 (Pin_1)
- net at J9.B5: now also P7.1 (Pin_1)
- net at J9.B8: now also P10.1 (Pin_1)
- net at J9.B9: now also P11.1 (Pin_1)
- net at J9.C11: now also P26.1 (Pin_1)
- net at J9.C12: now also P27.1 (Pin_1)
- net at J9.C13: now also P28.1 (Pin_1)
- net at J9.C14: now also P29.1 (Pin_1)
- net at J9.C16: now also P30.1 (Pin_1)
- net at J9.C26: now also P31.1 (Pin_1)
- net at J9.C3: now also P22.1 (Pin_1)
- net at J9.C39: now also P32.1 (Pin_1)
- net at J9.C4: now also P23.1 (Pin_1)
- net at J9.C50: now also P34.1 (Pin_1)
- net at J9.C6: now also P24.1 (Pin_1)
- net at J9.C9: now also P25.1 (Pin_1)
- net at J9.D1: now also P36.1 (Pin_1)
- net at J9.D11: now also P41.1 (Pin_1)
- net at J9.D15: now also P42.1 (Pin_1)
- net at J9.D16: now also P43.1 (Pin_1)
- net at J9.D19: now also P46.1 (Pin_1)
- net at J9.D2: now also P37.1 (Pin_1)
- net at J9.D21: now also P48.1 (Pin_1)
- net at J9.D25: now also P50.1 (Pin_1)
- net at J9.D27: now also P51.1 (Pin_1)
- net at J9.D29: now also P52.1 (Pin_1)
- net at J9.D31: now also P54.1 (Pin_1)
- net at J9.D34: now also P57.1 (Pin_1)
- net at J9.D35: now also P58.1 (Pin_1)
- net at J9.D40: now also P60.1 (Pin_1)
- net at J9.D5: now also P39.1 (Pin_1)
- net at J9.D6: now also P40.1 (Pin_1)
- net at J9.E4: now also P62.1 (Pin_1)
- net at J9.E8: now also P61.1 (Pin_1)
- net OUT_EXHAUST_FLAP_VALVE: no longer names the net of J9.D18
- net OUT_EXHAUST_FLAP_VALVE: now also P45.1 (Pin_1)
- net OUT_VANOS_INLET renamed OUT_VANOS_INTAKE
- net OUT_VANOS_INTAKE: now also BRD1.A20(16) (LS10(INJ10)), D1.2 (A)
- net OUT_VANOS_OTLET renamed OUT_VANOS_EXHAUST
- net OUT_VANOS_EXHAUST: now also BRD1.A9(4) (LS11(INJ11)), D2.2 (A)
- new net SEC_AIR_PUMP_RELAY: BRD1.A25(34) (IGN12), Q7.1 (IN), R16.2
- no-connect marks 57 -> 17

Commit message: Upd pcb
Parts:
- added G1: RUSEFI_LOGO, kicad6-libraries:rusefi_logo, symbol rusefi_logo:RUSEFI_LOGO
- added G2, G3, G4, G5, G6, G7, G8: PROTO_AREA, hellen-one-common:PROTO_AREA, symbol hellen-one-common:PROTO_AREA
- added J7: Conn_01x01, TestPoint:TestPoint_Pad_D4.0mm, symbol Connector_Generic:Conn_01x01
- added P63, P64, P65, P66, P67, P68, P69, P70, P71, P72, P73, P74, P75, P76, P77, P78, P79, P80, P81, P82, P83: Pad, hellen-one-common:PAD-TH, symbol hellen-one-common:Pad
Connections:
- net +5VA: now also G6.10, G6.6, G6.7, G6.8, G6.9
- net GND: now also G6.1, G6.2, G6.3, G6.4, G6.5, J7.1 (Pin_1)
- net at BRD1.A1(12) (HS2): now also P65.1 (Pin_1)
- net at BRD1.A13(23) (HS3): now also P66.1 (Pin_1)
- net at BRD1.A14(22) (HS4): now also P67.1 (Pin_1)
- net at BRD1.A2(11) (HS1): now also P64.1 (Pin_1)
- net at BRD1.A26(33) (IGN11): now also P71.1 (Pin_1)
- net at BRD1.A27(32) (IGN10): now also P63.1 (Pin_1)
- net at BRD1.A28(31) (IGN9): now also P70.1 (Pin_1)
- net at BRD1.A29(30) (IGN8): now also P69.1 (Pin_1)
- net at BRD1.A30(29) (IGN7): now also P68.1 (Pin_1)
- net at BRD1.B12(12) (VR2-): now also P75.1 (Pin_1)
- net at BRD1.B13(11) (VR1-): now also P73.1 (Pin_1)
- net at BRD1.B15(9) (ETB2+): now also P76.1 (Pin_1)
- net at BRD1.B4(5) (VR2+): now also P74.1 (Pin_1)
- net at BRD1.B5(4) (VR1+): now also P72.1 (Pin_1)
- net at BRD1.B8(1) (ETB2-): now also P77.1 (Pin_1)
- net at BRD1.C10(3) (5V_2): now also BRD1.C22(14) (5V_2), BRD1.C33(26) (5V_2), P83.1 (Pin_1)
- net 12V_PROT: now reaches BRD1.C11(2) (12V_PROT)
- net 12V_PROT: now also BRD1.C12(1) (12V_PROT), G6.11, G6.12, G6.13, G6.14, G6.15
- net at BRD1.C17(19) (AV9): now also P79.1 (Pin_1)
- net at BRD1.C18(18) (AV11): now also P81.1 (Pin_1)
- net at BRD1.C27(32) (AV8): now also P78.1 (Pin_1)
- net at BRD1.C28(31) (AV10): now also P80.1 (Pin_1)
- net at BRD1.C31(28) (AT4): now also P82.1 (Pin_1)
- new net: G4.1, G4.11, G4.6
- new net: G4.10, G4.15, G4.5
- new net: G4.12, G4.2, G4.7
- new net: G4.13, G4.3, G4.8
- new net: G4.14, G4.4, G4.9
- new net: G7.1, G7.11, G7.6
- new net: G7.10, G7.15, G7.5
- new net: G7.12, G7.2, G7.7
- new net: G7.13, G7.3, G7.8
- new net: G7.14, G7.4, G7.9
- new net: G3.1, G3.11, G3.6
- new net: G3.10, G3.15, G3.5
- new net: G3.12, G3.2, G3.7
- new net: G3.13, G3.3, G3.8
- new net: G3.14, G3.4, G3.9
- new net: G2.1, G2.11, G2.6
- new net: G2.10, G2.15, G2.5
- new net: G2.12, G2.2, G2.7
- new net: G2.13, G2.3, G2.8
- new net: G2.14, G2.4, G2.9
- new net: G5.1, G5.11, G5.6
- new net: G5.10, G5.15, G5.5
- new net: G5.12, G5.2, G5.7
- new net: G5.13, G5.3, G5.8
- new net: G5.14, G5.4, G5.9
- new net: G8.1, G8.11, G8.6
- new net: G8.10, G8.15, G8.5
- new net: G8.12, G8.2, G8.7
- new net: G8.13, G8.3, G8.8
- new net: G8.14, G8.4, G8.9
Other:
- note removed: "??"

Commit message: Fab preview
Parts:
- removed J6: Conn_01x01, MountingHole:MountingHole_4.5mm, symbol Connector_Generic:Conn_01x01
Connections:
- no-connect marks 17 -> 21
Other:
- note removed: "TODO: Add "baro" silkscreen"
- moved on the sheet: BRD1, C1, C2, C3, C4, F3, F4, F5, F6, F7, F8, J10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
